File: LT3758-Test-HW.kicad_pcb (KiCad board)
At the start: 2 copper layers, 50 x 25 mm, 27 parts, among them J1 Pins_2.54_1x2, J2 Pins_2.54_1x2, Q1 AON2290, U1 LT3758EDD

Commit message: Add text block
Other:
- board text added: "LT3758-Test v1.0 Jul 23"
Changed lines of the file:
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@@
   (gr_rect (start 46.7 38.5) (end 96.7 63.5)
     (stroke (width 0.1) (type default)) (fill none) (layer "Edge.Cuts"))
+  (gr_text "LT3758-Test\nv1.0\nJul 23" (at 94.5 44.4) (layer "B.SilkS")
+    (effects (font (size 1 1) (thickness 0.15)) (justify left bottom mirror))
+  )
   (gr_text "VOUT" (at 89.5 57.7) (layer "F.SilkS" knockout)
     (effects (font (size 1.5 1.5) (thickness 0.3) bold) (justify left bottom))
